Commit message: porting
porting from local

File: urdf/olive_grove_geometry.urdf.xacro (robot description, xacro)
@@ -25,4 +25,10 @@
       </geometry>
     </visual>
+    <visual>
+      <origin xyz="-35 -37 0" rpy="0 0 0"/>
+      <geometry>
+        <mesh filename="package://olive_grove_gazebo/meshes/arrow.dae"/>
+      </geometry>
+    </visual>
     <collision>
       <origin xyz="0 0 0" rpy="0 0 1.5707963267948966"/>
@@ -45,4 +51,16 @@
       </geometry>
     </collision>
+    <collision>
+      <origin xyz="0 0 0" rpy="0 0 1.5707963267948966"/>
+      <geometry>
+        <mesh filename="package://olive_grove_gazebo/meshes/leaves_grove.dae"/>
+      </geometry>
+    </collision>
+    <collision>
+      <origin xyz="-35 -37 0" rpy="0 0 0"/>
+      <geometry>
+        <mesh filename="package://olive_grove_gazebo/meshes/arrow.dae"/>
+      </geometry>
+    </collision>
   </link>
   <gazebo> <static>true</static></gazebo>
